File: PCBs/pic18f_DB_Ethernet.sch (KiCad schematic (older format))
At the start: 32 parts, among them J1 OC1, J2 PicKIT 3, J3 IC1, J4 FC1, J5 MC1, J6 DB9_Female, J7 DB9_Male, J8 RJ45, SW1 SW_DPDT_x2, SW2 PWR_SW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

Commit message: Added dpdt switch from stock. added battery clip. Reconsidering mouser bites. TODO: Orthagonal repo of parts rendered in KiCAD.
Parts:
- added unit 2 of SW2
- BT1: footprint (none) -> BAT-HLD-001:BAT-HLD-001
- SW1, SW2: footprint (none) -> JS202011SCQN:JS202011SCQN
Connections:
- net 3v3: now also SW2.6 (C)
- net at BT1.1 (+), SW2.2 (B): now also SW2.5 (B)
- no-connect marks 1 -> 2
Changed lines of the file:
@@
 F 0 "BT1" H 1718 2196 50  0000 L CNN
 F 1 "CR2032" H 1718 2105 50  0000 L CNN
-F 2 "" V 1600 2160 50  0001 C CNN
+F 2 "BAT-HLD-001:BAT-HLD-001" V 1600 2160 50  0001 C CNN
 F 3 "~" V 1600 2160 50  0001 C CNN
 	1    1600 2100
@@
 F 0 "SW2" H 1950 1835 50  0000 C CNN
 F 1 "PWR_SW" H 1950 1744 50  0000 C CNN
-F 2 "" H 1950 1550 50  0001 C CNN
+F 2 "JS202011SCQN:JS202011SCQN" H 1950 1550 50  0001 C CNN
 F 3 "" H 1950 1550 50  0001 C CNN
 	1    1950 1550
@@
 F 0 "SW1" H 1800 3485 50  0000 C CNN
 F 1 "SW_DPDT_x2" H 1800 3394 50  0000 C CNN
-F 2 "" H 1800 3200 50  0001 C CNN
+F 2 "JS202011SCQN:JS202011SCQN" H 1800 3200 50  0001 C CNN
 F 3 "" H 1800 3200 50  0001 C CNN
 	1    1800 3200
@@
 F 0 "SW1" H 1800 4335 50  0000 C CNN
 F 1 "SW_DPDT_x2" H 1800 4244 50  0000 C CNN
-F 2 "" H 1800 4050 50  0001 C CNN
+F 2 "JS202011SCQN:JS202011SCQN" H 1800 4050 50  0001 C CNN
 F 3 "" H 1800 4050 50  0001 C CNN
 	2    1800 4050
@@
 	2250 3300 2150 3300
 Connection ~ 2150 3300
+$Comp
+L Switch:SW_DPDT_x2 SW2
+U 2 1 5E647F5E
+P 3000 1550
+F 0 "SW2" H 3000 1835 50  0000 C CNN
+F 1 "PWR_SW" H 3000 1744 50  0000 C CNN
+F 2 "" H 3000 1550 50  0001 C CNN
+F 3 "" H 3000 1550 50  0001 C CNN
+	2    3000 1550
+	1    0    0    -1
+$EndComp
+NoConn ~ 3200 1450
+Wire Wire Line
+	2800 1550 2650 1550
+Wire Wire Line
+	2650 1550 2650 1100
+Wire Wire Line
+	2650 1100 1600 1100
+Wire Wire Line
+	1600 1100 1600 1550
+Connection ~ 1600 1550
+Wire Wire Line
+	2150 1650 2150 1850
+Wire Wire Line
+	2150 1850 3200 1850
+Wire Wire Line
+	3200 1850 3200 1650
+Connection ~ 2150 1650
 $EndSCHEMATC

Commit message: Finished Rev A layout. Some research revealed that JLCPCB does not support what I want. I might just send the break out into a different pcb.
Parts:
- added H1, H2, H3, H4, H5, H6, H7, H8: MountingHole, MountingHole:MountingHole_3.2mm_M3, symbol Mechanical:MountingHole
- SW2: footprint (none) -> JS202011SCQN:JS202011SCQN
Changed lines of the file:
@@
 F 0 "SW2" H 3000 1835 50  0000 C CNN
 F 1 "PWR_SW" H 3000 1744 50  0000 C CNN
-F 2 "" H 3000 1550 50  0001 C CNN
+F 2 "JS202011SCQN:JS202011SCQN" H 3000 1550 50  0001 C CNN
 F 3 "" H 3000 1550 50  0001 C CNN
 	2    3000 1550
@@
 	3200 1850 3200 1650
 Connection ~ 2150 1650
+$Comp
+L Mechanical:MountingHole H1
+U 1 1 5E67B493
+P 1100 6050
+F 0 "H1" H 1200 6096 50  0000 L CNN
+F 1 "MountingHole" H 1200 6005 50  0000 L CNN
+F 2 "MountingHole:MountingHole_3.2mm_M3" H 1100 6050 50  0001 C CNN
+F 3 "~" H 1100 6050 50  0001 C CNN
+	1    1100 6050
+	1    0    0    -1
+$EndComp
+$Comp
+L Mechanical:MountingHole H2
+U 1 1 5E67B591
+P 1100 6300
+F 0 "H2" H 1200 6346 50  0000 L CNN
+F 1 "MountingHole" H 1200 6255 50  0000 L CNN
+F 2 "MountingHole:MountingHole_3.2mm_M3" H 1100 6300 50  0001 C CNN
+F 3 "~" H 1100 6300 50  0001 C CNN
+	1    1100 6300
+	1    0    0    -1
+$EndComp
+$Comp
+L Mechanical:MountingHole H3
+U 1 1 5E686EAD
+P 1100 6550
+F 0 "H3" H 1200 6596 50  0000 L CNN
+F 1 "MountingHole" H 1200 6505 50  0000 L CNN
+F 2 "MountingHole:MountingHole_3.2mm_M3" H 1100 6550 50  0001 C CNN
+F 3 "~" H 1100 6550 50  0001 C CNN
+	1    1100 6550
+	1    0    0    -1
+$EndComp
+$Comp
+L Mechanical:MountingHole H4
+U 1 1 5E69265C
+P 1100 6800
+F 0 "H4" H 1200 6846 50  0000 L CNN
+F 1 "MountingHole" H 1200 6755 50  0000 L CNN
+F 2 "MountingHole:MountingHole_3.2mm_M3" H 1100 6800 50  0001 C CNN
+F 3 "~" H 1100 6800 50  0001 C CNN
+	1    1100 6800
+	1    0    0    -1
+$EndComp
+$Comp
+L Mechanical:MountingHole H5
+U 1 1 5E69DF10
+P 1950 6050
+F 0 "H5" H 2050 6096 50  0000 L CNN
+F 1 "MountingHole" H 2050 6005 50  0000 L CNN
+F 2 "MountingHole:MountingHole_3.2mm_M3" H 1950 6050 50  0001 C CNN
+F 3 "~" H 1950 6050 50  0001 C CNN
+	1    1950 6050
+	1    0    0    -1
+$EndComp
+$Comp
+L Mechanical:MountingHole H6
+U 1 1 5E69DF17
+P 1950 6300
+F 0 "H6" H 2050 6346 50  0000 L CNN
+F 1 "MountingHole" H 2050 6255 50  0000 L CNN
+F 2 "MountingHole:MountingHole_3.2mm_M3" H 1950 6300 50  0001 C CNN
+F 3 "~" H 1950 6300 50  0001 C CNN
+	1    1950 6300
+	1    0    0    -1
+$EndComp
+$Comp
+L Mechanical:MountingHole H7
+U 1 1 5E69DF1E
+P 1950 6550
+F 0 "H7" H 2050 6596 50  0000 L CNN
+F 1 "MountingHole" H 2050 6505 50  0000 L CNN
+F 2 "MountingHole:MountingHole_3.2mm_M3" H 1950 6550 50  0001 C CNN
+F 3 "~" H 1950 6550 50  0001 C CNN
+	1    1950 6550
+	1    0    0    -1
+$EndComp
+$Comp
+L Mechanical:MountingHole H8
+U 1 1 5E69DF25
+P 1950 6800
+F 0 "H8" H 2050 6846 50  0000 L CNN
+F 1 "MountingHole" H 2050 6755 50  0000 L CNN
+F 2 "MountingHole:MountingHole_3.2mm_M3" H 1950 6800 50  0001 C CNN
+F 3 "~" H 1950 6800 50  0001 C CNN
+	1    1950 6800
+	1    0    0    -1
+$EndComp
 $EndSCHEMATC

Commit message: Restructed project
Parts:
- removed H5, H6, H7, H8: MountingHole, MountingHole:MountingHole_3.2mm_M3, symbol Mechanical:MountingHole
- removed J4: FC1, Connector_PinHeader_2.54mm:PinHeader_2x05_P2.54mm_Vertical, symbol Connector_Generic:Conn_02x05_Odd_Even
- removed J5: MC1, Connector_PinHeader_2.54mm:PinHeader_2x05_P2.54mm_Vertical, symbol Connector_Generic:Conn_02x05_Odd_Even
- removed J6: DB9_Female, Connector_Dsub:DSUB-9_Female_Horizontal_P2.77x2.84mm_EdgePinOffset9.90mm_Housed_MountingHolesOffset11.32mm, symbol Connector:DB9_Female
- removed J7: DB9_Male, Connector_Dsub:DSUB-9_Female_Horizontal_P2.77x2.84mm_EdgePinOffset9.90mm_Housed_MountingHolesOffset11.32mm, symbol Connector:DB9_Male
Other:
- moved on the sheet: D1, D10, D2, D3, D4, D5, D6, D7, D8, D9, H1, H2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

Commit message: changed RJ45 jack to unsheilded. Printed main board gerbers and gerber pdfs
Parts:
- J8: footprint Connector_RJ:RJ45_Amphenol_RJHSE5380 -> Connector_RJ:RJ45_Amphenol_54602-x08_Horizontal
Changed lines of the file:
@@
 F 0 "J8" H 8520 1204 50  0000 R CNN
 F 1 "RJ45" H 8520 1295 50  0000 R CNN
-F 2 "Connector_RJ:RJ45_Amphenol_RJHSE5380" V 8850 1225 50  0001 C CNN
+F 2 "Connector_RJ:RJ45_Amphenol_54602-x08_Horizontal" V 8850 1225 50  0001 C CNN
 F 3 "~" V 8850 1225 50  0001 C CNN
 	1    8850 1200
